File: node-mcu-pack.brd (EAGLE design)
At the start: 25.5 x 48 mm, 10 parts, among them J1 IOBLOCK6, J2 IOBLOCK6, U1 L9110SMT, U2 L9110SMT

Commit message: moved i2c pins for wiicuck
Connections:
- removed net N$13: J1.P$3, U$1.D2
- new net D2: J1.P$3, U$1.D2, U$2.DAT
- net D0: no longer U$2.CLK
- net D1: now also U$2.CLK; no longer U$2.DAT
Routing:
- net D2: track 0.00 -> 23.7 mm
- net D0: track 21.1 -> 3.16 mm
- net D1: track 18.6 -> 23.9 mm
- net N$13: track 3.16 -> 0.00 mm
Changed lines of the file:
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@@
 <wire x1="39.38" y1="34.21" x2="39.43" y2="34.16" width="0.4064" layer="1"/>
-</signal>
-<signal name="N$13">
-<contactref element="U$1" pad="D2"/>
-<contactref element="J1" pad="P$3"/>
-<wire x1="36.29" y1="36.75" x2="39.38" y2="36.75" width="0.4064" layer="1"/>
-<wire x1="39.38" y1="36.75" x2="39.43" y2="36.7" width="0.4064" layer="1"/>
 </signal>
 <signal name="3V3">
@@
 <wire x1="34.8" y1="30.3" x2="33.2" y2="30.3" width="0.1524" layer="16"/>
 <wire x1="33.2" y1="30.3" x2="32.55" y2="30.95" width="0.1524" layer="16"/>
-<wire x1="32.55" y1="30.95" x2="32.55" y2="44.15" width="0.1524" layer="16"/>
-<wire x1="32.55" y1="44.15" x2="30.75" y2="45.95" width="0.1524" layer="16"/>
+<wire x1="32.55" y1="30.95" x2="32.55" y2="42.8" width="0.1524" layer="16"/>
 <wire x1="25.745" y1="47.85" x2="25.745" y2="52.2" width="0.1524" layer="16"/>
-<wire x1="30.75" y1="45.95" x2="30.75" y2="46.75" width="0.1524" layer="16"/>
-<wire x1="30.75" y1="46.75" x2="29.8" y2="47.7" width="0.1524" layer="16"/>
-<wire x1="29.8" y1="47.7" x2="25.895" y2="47.7" width="0.1524" layer="16"/>
-<wire x1="25.895" y1="47.7" x2="25.745" y2="47.85" width="0.1524" layer="16"/>
+<wire x1="25.745" y1="47.85" x2="25.745" y2="45.755" width="0.254" layer="16"/>
+<wire x1="25.745" y1="45.755" x2="27.8" y2="43.7" width="0.254" layer="16"/>
+<wire x1="27.8" y1="43.7" x2="31.65" y2="43.7" width="0.254" layer="16"/>
+<wire x1="31.65" y1="43.7" x2="32.55" y2="42.8" width="0.254" layer="16"/>
 </signal>
 <signal name="D1">
-<contactref element="U$2" pad="DAT"/>
 <contactref element="U$1" pad="D1"/>
 <contactref element="J1" pad="P$2"/>
 <wire x1="36.29" y1="39.29" x2="39.38" y2="39.29" width="0.4064" layer="1"/>
 <wire x1="39.38" y1="39.29" x2="39.43" y2="39.24" width="0.4064" layer="1"/>
-<wire x1="36.29" y1="39.29" x2="35.05" y2="40.53" width="0.1524" layer="16"/>
-<wire x1="35.05" y1="40.53" x2="35.05" y2="43.05" width="0.1524" layer="16"/>
-<wire x1="35.05" y1="43.05" x2="30.255" y2="47.845" width="0.1524" layer="16"/>
-<wire x1="30.255" y1="47.845" x2="30.255" y2="52.2" width="0.1524" layer="16"/>
+<contactref element="U$2" pad="CLK"/>
+<wire x1="25.745" y1="52.2" x2="25.745" y2="47.455" width="0.254" layer="1"/>
+<wire x1="25.745" y1="47.455" x2="28.1" y2="45.1" width="0.254" layer="1"/>
+<wire x1="28.1" y1="45.1" x2="33.3" y2="45.1" width="0.254" layer="1"/>
+<wire x1="33.3" y1="45.1" x2="35" y2="43.4" width="0.254" layer="1"/>
+<wire x1="35" y1="43.4" x2="35" y2="39.8" width="0.254" layer="1"/>
+<wire x1="35" y1="39.8" x2="35.51" y2="39.29" width="0.254" layer="1"/>
+<wire x1="35.51" y1="39.29" x2="36.29" y2="39.29" width="0.254" layer="1"/>
 </signal>
 <signal name="D0">
-<contactref element="U$2" pad="CLK"/>
 <contactref element="U$1" pad="D0"/>
 <contactref element="J1" pad="P$1"/>
 <wire x1="36.29" y1="41.83" x2="39.38" y2="41.83" width="0.4064" layer="1"/>
 <wire x1="39.38" y1="41.83" x2="39.43" y2="41.78" width="0.4064" layer="1"/>
-<wire x1="36.29" y1="41.83" x2="36.29" y2="42.96" width="0.1524" layer="1"/>
-<wire x1="25.85" y1="48" x2="25.85" y2="51.3" width="0.1524" layer="1"/>
-<wire x1="25.85" y1="51.3" x2="25.745" y2="51.405" width="0.1524" layer="1"/>
-<wire x1="25.745" y1="51.405" x2="25.745" y2="52.2" width="0.1524" layer="1"/>
-<wire x1="36.29" y1="42.96" x2="34.2" y2="45.05" width="0.1524" layer="1"/>
-<wire x1="34.2" y1="45.05" x2="28.8" y2="45.05" width="0.1524" layer="1"/>
-<wire x1="28.8" y1="45.05" x2="25.85" y2="48" width="0.1524" layer="1"/>
 </signal>
 <signal name="1BO">
@@
 <wire x1="34.35" y1="6.5" x2="35.3" y2="7.45" width="1.016" layer="1"/>
 </signal>
+<signal name="D2">
+<contactref element="U$2" pad="DAT"/>
+<contactref element="U$1" pad="D2"/>
+<contactref element="J1" pad="P$3"/>
+<wire x1="36.29" y1="36.75" x2="39.38" y2="36.75" width="0.4064" layer="1"/>
+<wire x1="39.38" y1="36.75" x2="39.43" y2="36.7" width="0.4064" layer="1"/>
+<wire x1="30.255" y1="52.2" x2="30.255" y2="47.645" width="0.254" layer="16"/>
+<wire x1="30.255" y1="47.645" x2="31.5" y2="46.4" width="0.254" layer="16"/>
+<wire x1="31.5" y1="46.4" x2="32.9" y2="46.4" width="0.254" layer="16"/>
+<wire x1="32.9" y1="46.4" x2="36.2" y2="43.1" width="0.254" layer="16"/>
+<wire x1="36.2" y1="43.1" x2="36.9" y2="43.1" width="0.254" layer="16"/>
+<wire x1="36.9" y1="43.1" x2="37.9" y2="42.1" width="0.254" layer="16"/>
+<wire x1="37.9" y1="42.1" x2="37.9" y2="38.36" width="0.254" layer="16"/>
+<wire x1="37.9" y1="38.36" x2="36.29" y2="36.75" width="0.254" layer="16"/>
+</signal>
 </signals>
