File: node-mcu-pack.sch (EAGLE design)
At the start: 10 parts, among them J1 IOBLOCK6, J2 IOBLOCK6, U1 L9110SMT, U2 L9110SMT

Commit message: moved i2c pins for wiicuck
Connections:
- removed net N$13: J1.P$3, U$1.D2
- new net D2: J1.P$3, U$1.D2, U$2.SDA
- net D0: no longer U$2.SCL
- net D1: now also U$2.SCL; no longer U$2.SDA
Changed lines of the file:
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@@
-</segment>
-</net>
-<net name="N$13" class="0">
-<segment>
-<pinref part="U$1" gate="G$1" pin="D2"/>
-<pinref part="J1" gate="G$1" pin="P$3"/>
-<wire x1="83.82" y1="66.04" x2="91.44" y2="66.04" width="0.1524" layer="91"/>
 </segment>
 </net>
@@
 <net name="D1" class="0">
 <segment>
-<pinref part="U$2" gate="G$1" pin="SDA"/>
-<wire x1="83.82" y1="96.52" x2="73.66" y2="96.52" width="0.1524" layer="91"/>
-<label x="73.66" y="96.52" size="1.27" layer="95" rot="R180" xref="yes"/>
-</segment>
-<segment>
 <pinref part="U$1" gate="G$1" pin="D1"/>
 <pinref part="J1" gate="G$1" pin="P$2"/>
 <wire x1="83.82" y1="68.58" x2="91.44" y2="68.58" width="0.1524" layer="91"/>
 </segment>
-</net>
-<net name="D0" class="0">
 <segment>
 <pinref part="U$2" gate="G$1" pin="SCL"/>
@@
 <label x="73.66" y="93.98" size="1.27" layer="95" rot="R180" xref="yes"/>
 </segment>
+</net>
+<net name="D0" class="0">
 <segment>
 <pinref part="U$1" gate="G$1" pin="D0"/>
@@
 </segment>
 </net>
+<net name="D2" class="0">
+<segment>
+<pinref part="U$2" gate="G$1" pin="SDA"/>
+<wire x1="83.82" y1="96.52" x2="73.66" y2="96.52" width="0.1524" layer="91"/>
+<label x="73.66" y="96.52" size="1.27" layer="95" rot="R180" xref="yes"/>
+</segment>
+<segment>
+<pinref part="U$1" gate="G$1" pin="D2"/>
+<pinref part="J1" gate="G$1" pin="P$3"/>
+<wire x1="83.82" y1="66.04" x2="91.44" y2="66.04" width="0.1524" layer="91"/>
+</segment>
+</net>
